Commit message: Refactor robot.urdf with updated inertial properties
Updated inertial properties for base link and adjusted dimensions for joints and links.

File: robot.urdf (robot description, URDF)
Before this commit: robot robo_dog, 13 links, 12 joints
Links:
- link FL_calf: geometry collision cylinder length=0.12 radius=0.01; visual cylinder length=0.12 radius=0.01
- link FL_thigh: geometry visual cylinder length=0.10 radius=0.015
- link FR_calf: geometry collision cylinder length=0.12 radius=0.01; visual cylinder length=0.12 radius=0.01
- link FR_thigh: geometry visual cylinder length=0.10 radius=0.015
- link RL_calf: geometry collision cylinder length=0.12 radius=0.01; visual cylinder length=0.12 radius=0.01
- link RL_thigh: geometry visual cylinder length=0.10 radius=0.015
- link RR_calf: geometry collision cylinder length=0.12 radius=0.01; visual cylinder length=0.12 radius=0.01
- link RR_thigh: geometry visual cylinder length=0.10 radius=0.015
Joints:
- joint FL_knee_joint: origin xyz=0 0 -0.12 rpy=0 0 0 -> xyz=0 0 -0.1 rpy=0 0 0
- joint FR_knee_joint: origin xyz=0 0 -0.12 rpy=0 0 0 -> xyz=0 0 -0.1 rpy=0 0 0
- joint RL_knee_joint: origin xyz=0 0 -0.12 rpy=0 0 0 -> xyz=0 0 -0.1 rpy=0 0 0
- joint RR_knee_joint: origin xyz=0 0 -0.12 rpy=0 0 0 -> xyz=0 0 -0.1 rpy=0 0 0
